Commit message: add dynamic & random static obstacles

File: assets/urdf/project_mobile_robot/lidar_sensor.urdf.xacro (robot description, xacro)
@@ -13,16 +13,4 @@
         <inertia ixx="0.000000017" ixy="0" ixz="0" iyy="0.000000017" iyz="0" izz="0.000000017" />
       </inertial>
-      <!--<visual>-->
-        <!--<origin xyz="0 0 0" rpy="0 0 0" />-->
-        <!--<geometry>-->
-          <!--<box size="0.01 0.01 0.01" /> -->
-        <!--</geometry>-->
-      <!--</visual>-->
-   <!--   <collision>
-        <origin xyz="0 0 0" rpy="0 0 0" />
-        <geometry>
-          <box size="0.01 0.01 0.01" />
-        </geometry>
-      </collision> -->
     </link>
     <gazebo reference="${name}_link">

File: assets/urdf/project_mobile_robot/project_mobile_robot.urdf.xacro (robot description, xacro)
@@ -18,5 +18,5 @@
     <visual>
       <geometry>
-        <cylinder length="0.3" radius="0.201"/>
+        <cylinder length="0.15" radius="0.201"/>
       </geometry>
       <material name="grey"/>
@@ -24,5 +24,5 @@
     <collision>
       <geometry>
-        <cylinder length="0.3" radius="0.201"/>
+        <cylinder length="0.15" radius="0.201"/>
       </geometry>
     </collision>
@@ -57,8 +57,8 @@
     </joint>
   </xacro:macro>
-  <xacro:wheel_link name="left" linkrpy="0 0 0" axisxyz="1 0 0" originxyz="0.15 0 -0.15"/>
-  <xacro:wheel_link name="right" linkrpy="0 0 0" axisxyz="1 0 0" originxyz="-0.15 0 -0.15"/>
-  <xacro:wheel_link name="front" linkrpy="0 0 0" axisxyz="0 1 0" originxyz="0 0.15 -0.15"/>
-  <xacro:wheel_link name="back" linkrpy="0 0 0" axisxyz="0 1 0" originxyz="0 -0.15 -0.15"/>
+  <xacro:wheel_link name="left" linkrpy="0 0 0" axisxyz="1 0 0" originxyz="0.15 0 -0.075"/>
+  <xacro:wheel_link name="right" linkrpy="0 0 0" axisxyz="1 0 0" originxyz="-0.15 0 -0.075"/>
+  <xacro:wheel_link name="front" linkrpy="0 0 0" axisxyz="0 1 0" originxyz="0 0.15 -0.075"/>
+  <xacro:wheel_link name="back" linkrpy="0 0 0" axisxyz="0 1 0" originxyz="0 -0.15 -0.075"/>
   <!-- Lidar sensor -->
   <xacro:include filename="lidar_sensor.urdf.xacro"/>
@@ -76,4 +76,5 @@
     ray_count_vertical="1">
     <origin xyz="0 0.0 0.17" rpy="0 0 0"/>
+    <!-- origin xyz="0 0.0 0.17" rpy="0 0 0"/-->
   </xacro:lidar_sensor>
   <gazebo>
