Commit message: upgrade dynamic obstacles

File: assets/urdf/project_mobile_robot/project_mobile_robot.urdf.xacro (robot description, xacro)
@@ -75,6 +75,5 @@
     ray_count_horizontal="216"
     ray_count_vertical="1">
-    <origin xyz="0 0.0 0.17" rpy="0 0 0"/>
-    <!-- origin xyz="0 0.0 0.17" rpy="0 0 0"/-->
+    <origin xyz="0 0.0 0.1" rpy="0 0 0"/>
   </xacro:lidar_sensor>
   <gazebo>

Commit message: actor_critic v0.2 and map changes

File: assets/urdf/project_mobile_robot/project_mobile_robot.urdf.xacro (robot description, xacro)
@@ -11,5 +11,5 @@
     <inertial>
       <mass value="${mass}"/>
-      <inertia ixx="1.0" ixy="0.0" ixz="0.0" iyy="1.0" iyz="0.0" izz="1.0"/>
+      <inertia ixx="${mass}" ixy="0.0" ixz="0.0" iyy="${mass}" iyz="0.0" izz="${mass}"/>
     </inertial>
   </xacro:macro>
@@ -48,5 +48,5 @@
         <origin xyz="0 0 0" rpy="${linkrpy}"/>
       </collision>
-      <xacro:default_inertial mass="1"/>
+      <xacro:default_inertial mass="1.0"/>
     </link>
     <joint name="${name}_wheel_joint" type="fixed">

Commit message: actor_critic v7.0
change learning algorithm, normalized, urdf test program, new robot model(axis changes)

File: assets/urdf/project_mobile_robot/project_mobile_robot.urdf.xacro (robot description, xacro)
@@ -57,8 +57,8 @@
     </joint>
   </xacro:macro>
-  <xacro:wheel_link name="left" linkrpy="0 0 0" axisxyz="1 0 0" originxyz="0.15 0 -0.075"/>
-  <xacro:wheel_link name="right" linkrpy="0 0 0" axisxyz="1 0 0" originxyz="-0.15 0 -0.075"/>
-  <xacro:wheel_link name="front" linkrpy="0 0 0" axisxyz="0 1 0" originxyz="0 0.15 -0.075"/>
-  <xacro:wheel_link name="back" linkrpy="0 0 0" axisxyz="0 1 0" originxyz="0 -0.15 -0.075"/>
+  <xacro:wheel_link name="front_right" linkrpy="0 0 0" axisxyz="1 0 0" originxyz="0.15 0 -0.075"/>
+  <xacro:wheel_link name="back_left" linkrpy="0 0 0" axisxyz="1 0 0" originxyz="-0.15 0 -0.075"/>
+  <xacro:wheel_link name="front_left" linkrpy="0 0 0" axisxyz="0 1 0" originxyz="0 0.15 -0.075"/>
+  <xacro:wheel_link name="back_right" linkrpy="0 0 0" axisxyz="0 1 0" originxyz="0 -0.15 -0.075"/>
   <!-- Lidar sensor -->
   <xacro:include filename="lidar_sensor.urdf.xacro"/>
@@ -75,5 +75,5 @@
     ray_count_horizontal="20"
     ray_count_vertical="1">
-    <origin xyz="0 0.0 0.1" rpy="0 0 0"/>
+    <origin xyz="0 0.0 0.1" rpy="0 0 ${M_PI/4}"/>
   </xacro:lidar_sensor>
   <gazebo>

Commit message: q_learning
environment setting

File: assets/urdf/project_mobile_robot/project_mobile_robot.urdf.xacro (robot description, xacro)
@@ -57,11 +57,11 @@
     </joint>
   </xacro:macro>
-  <xacro:wheel_link name="front_right" linkrpy="0 0 0" axisxyz="1 0 0" originxyz="0.15 0 -0.075"/>
-  <xacro:wheel_link name="back_left" linkrpy="0 0 0" axisxyz="1 0 0" originxyz="-0.15 0 -0.075"/>
-  <xacro:wheel_link name="front_left" linkrpy="0 0 0" axisxyz="0 1 0" originxyz="0 0.15 -0.075"/>
-  <xacro:wheel_link name="back_right" linkrpy="0 0 0" axisxyz="0 1 0" originxyz="0 -0.15 -0.075"/>
+  <xacro:wheel_link name="left" linkrpy="0 0 0" axisxyz="1 0 0" originxyz="0.15 0 -0.075"/>
+  <xacro:wheel_link name="right" linkrpy="0 0 0" axisxyz="1 0 0" originxyz="-0.15 0 -0.075"/>
+  <xacro:wheel_link name="front" linkrpy="0 0 0" axisxyz="0 1 0" originxyz="0 0.15 -0.075"/>
+  <xacro:wheel_link name="back" linkrpy="0 0 0" axisxyz="0 1 0" originxyz="0 -0.15 -0.075"/>
   <!-- Lidar sensor -->
   <xacro:include filename="lidar_sensor.urdf.xacro"/>
-  <!--Q:ray_count_horizontal=60, DQN:ray_count_horizontal=216 -->
+  <!--Q:ray_count_horizontal=10, DQN:ray_count_horizontal=216 -->
   <xacro:lidar_sensor
     name="sonar"
@@ -73,7 +73,7 @@
     field_of_view_horizontal="${270*M_PI/180}"
     field_of_view_vertical="${1*M_PI/180}"
-    ray_count_horizontal="20"
+    ray_count_horizontal="2160"
     ray_count_vertical="1">
-    <origin xyz="0 0.0 0.1" rpy="0 0 ${M_PI/4}"/>
+    <origin xyz="0 0.0 0.1" rpy="0 0 0"/>
   </xacro:lidar_sensor>
   <gazebo>

Commit message: actor_critic

File: assets/urdf/project_mobile_robot/project_mobile_robot.urdf.xacro (robot description, xacro)
@@ -57,11 +57,11 @@
     </joint>
   </xacro:macro>
-  <xacro:wheel_link name="left" linkrpy="0 0 0" axisxyz="1 0 0" originxyz="0.15 0 -0.075"/>
-  <xacro:wheel_link name="right" linkrpy="0 0 0" axisxyz="1 0 0" originxyz="-0.15 0 -0.075"/>
-  <xacro:wheel_link name="front" linkrpy="0 0 0" axisxyz="0 1 0" originxyz="0 0.15 -0.075"/>
-  <xacro:wheel_link name="back" linkrpy="0 0 0" axisxyz="0 1 0" originxyz="0 -0.15 -0.075"/>
+  <xacro:wheel_link name="front_right" linkrpy="0 0 0" axisxyz="1 0 0" originxyz="0.15 0 -0.075"/>
+  <xacro:wheel_link name="back_left" linkrpy="0 0 0" axisxyz="1 0 0" originxyz="-0.15 0 -0.075"/>
+  <xacro:wheel_link name="front_left" linkrpy="0 0 0" axisxyz="0 1 0" originxyz="0 0.15 -0.075"/>
+  <xacro:wheel_link name="back_right" linkrpy="0 0 0" axisxyz="0 1 0" originxyz="0 -0.15 -0.075"/>
   <!-- Lidar sensor -->
   <xacro:include filename="lidar_sensor.urdf.xacro"/>
-  <!--Q:ray_count_horizontal=10, DQN:ray_count_horizontal=216 -->
+  <!--Q:ray_count_horizontal=60, DQN:ray_count_horizontal=216 -->
   <xacro:lidar_sensor
     name="sonar"
@@ -73,7 +73,7 @@
     field_of_view_horizontal="${270*M_PI/180}"
     field_of_view_vertical="${1*M_PI/180}"
-    ray_count_horizontal="2160"
+    ray_count_horizontal="20"
     ray_count_vertical="1">
-    <origin xyz="0 0.0 0.1" rpy="0 0 0"/>
+    <origin xyz="0 0.0 0.1" rpy="0 0 ${M_PI/4}"/>
   </xacro:lidar_sensor>
   <gazebo>

Commit message: q_learning new algo for states

File: assets/urdf/project_mobile_robot/project_mobile_robot.urdf.xacro (robot description, xacro)
@@ -57,11 +57,11 @@
     </joint>
   </xacro:macro>
-  <xacro:wheel_link name="front_right" linkrpy="0 0 0" axisxyz="1 0 0" originxyz="0.15 0 -0.075"/>
-  <xacro:wheel_link name="back_left" linkrpy="0 0 0" axisxyz="1 0 0" originxyz="-0.15 0 -0.075"/>
-  <xacro:wheel_link name="front_left" linkrpy="0 0 0" axisxyz="0 1 0" originxyz="0 0.15 -0.075"/>
-  <xacro:wheel_link name="back_right" linkrpy="0 0 0" axisxyz="0 1 0" originxyz="0 -0.15 -0.075"/>
+  <xacro:wheel_link name="left" linkrpy="0 0 0" axisxyz="1 0 0" originxyz="0.15 0 -0.075"/>
+  <xacro:wheel_link name="right" linkrpy="0 0 0" axisxyz="1 0 0" originxyz="-0.15 0 -0.075"/>
+  <xacro:wheel_link name="front" linkrpy="0 0 0" axisxyz="0 1 0" originxyz="0 0.15 -0.075"/>
+  <xacro:wheel_link name="back" linkrpy="0 0 0" axisxyz="0 1 0" originxyz="0 -0.15 -0.075"/>
   <!-- Lidar sensor -->
   <xacro:include filename="lidar_sensor.urdf.xacro"/>
-  <!--Q:ray_count_horizontal=60, DQN:ray_count_horizontal=216 -->
+  <!--Q:ray_count_horizontal=10, DQN:ray_count_horizontal=216 -->
   <xacro:lidar_sensor
     name="sonar"
@@ -73,7 +73,7 @@
     field_of_view_horizontal="${270*M_PI/180}"
     field_of_view_vertical="${1*M_PI/180}"
-    ray_count_horizontal="20"
+    ray_count_horizontal="2162"
     ray_count_vertical="1">
-    <origin xyz="0 0.0 0.1" rpy="0 0 ${M_PI/4}"/>
+    <origin xyz="0 0.0 0.1" rpy="0 0 0"/>
   </xacro:lidar_sensor>
   <gazebo>

Commit message: actor critic dynamic environment

File: assets/urdf/project_mobile_robot/project_mobile_robot.urdf.xacro (robot description, xacro)
@@ -57,11 +57,11 @@
     </joint>
   </xacro:macro>
-  <xacro:wheel_link name="left" linkrpy="0 0 0" axisxyz="1 0 0" originxyz="0.15 0 -0.075"/>
-  <xacro:wheel_link name="right" linkrpy="0 0 0" axisxyz="1 0 0" originxyz="-0.15 0 -0.075"/>
-  <xacro:wheel_link name="front" linkrpy="0 0 0" axisxyz="0 1 0" originxyz="0 0.15 -0.075"/>
-  <xacro:wheel_link name="back" linkrpy="0 0 0" axisxyz="0 1 0" originxyz="0 -0.15 -0.075"/>
+  <xacro:wheel_link name="front_right" linkrpy="0 0 0" axisxyz="1 0 0" originxyz="0.15 0 -0.075"/>
+  <xacro:wheel_link name="back_left" linkrpy="0 0 0" axisxyz="1 0 0" originxyz="-0.15 0 -0.075"/>
+  <xacro:wheel_link name="front_left" linkrpy="0 0 0" axisxyz="0 1 0" originxyz="0 0.15 -0.075"/>
+  <xacro:wheel_link name="back_right" linkrpy="0 0 0" axisxyz="0 1 0" originxyz="0 -0.15 -0.075"/>
   <!-- Lidar sensor -->
   <xacro:include filename="lidar_sensor.urdf.xacro"/>
-  <!--Q:ray_count_horizontal=10, DQN:ray_count_horizontal=216 -->
+  <!--Q:ray_count_horizontal=60, DQN:ray_count_horizontal=216 -->
   <xacro:lidar_sensor
     name="sonar"
@@ -73,7 +73,7 @@
     field_of_view_horizontal="${270*M_PI/180}"
     field_of_view_vertical="${1*M_PI/180}"
-    ray_count_horizontal="2162"
+    ray_count_horizontal="542"
     ray_count_vertical="1">
-    <origin xyz="0 0.0 0.1" rpy="0 0 0"/>
+    <origin xyz="0 0.0 0.1" rpy="0 0 ${M_PI/4}"/>
   </xacro:lidar_sensor>
   <gazebo>

Commit message: q learning map 2 program
median

File: assets/urdf/project_mobile_robot/project_mobile_robot.urdf.xacro (robot description, xacro)
@@ -57,11 +57,11 @@
     </joint>
   </xacro:macro>
-  <xacro:wheel_link name="front_right" linkrpy="0 0 0" axisxyz="1 0 0" originxyz="0.15 0 -0.075"/>
-  <xacro:wheel_link name="back_left" linkrpy="0 0 0" axisxyz="1 0 0" originxyz="-0.15 0 -0.075"/>
-  <xacro:wheel_link name="front_left" linkrpy="0 0 0" axisxyz="0 1 0" originxyz="0 0.15 -0.075"/>
-  <xacro:wheel_link name="back_right" linkrpy="0 0 0" axisxyz="0 1 0" originxyz="0 -0.15 -0.075"/>
+  <xacro:wheel_link name="left" linkrpy="0 0 0" axisxyz="1 0 0" originxyz="0.15 0 -0.075"/>
+  <xacro:wheel_link name="right" linkrpy="0 0 0" axisxyz="1 0 0" originxyz="-0.15 0 -0.075"/>
+  <xacro:wheel_link name="front" linkrpy="0 0 0" axisxyz="0 1 0" originxyz="0 0.15 -0.075"/>
+  <xacro:wheel_link name="back" linkrpy="0 0 0" axisxyz="0 1 0" originxyz="0 -0.15 -0.075"/>
   <!-- Lidar sensor -->
   <xacro:include filename="lidar_sensor.urdf.xacro"/>
-  <!--Q:ray_count_horizontal=60, DQN:ray_count_horizontal=216 -->
+  <!--Q:ray_count_horizontal=10, DQN:ray_count_horizontal=216 -->
   <xacro:lidar_sensor
     name="sonar"
@@ -73,7 +73,7 @@
     field_of_view_horizontal="${270*M_PI/180}"
     field_of_view_vertical="${1*M_PI/180}"
-    ray_count_horizontal="62"
+    ray_count_horizontal="2162"
     ray_count_vertical="1">
-    <origin xyz="0 0.0 0.1" rpy="0 0 ${M_PI/4}"/>
+    <origin xyz="0 0.0 0.1" rpy="0 0 0"/>
   </xacro:lidar_sensor>
   <gazebo>

Commit message: 105 states, 3x20 map, new reward

File: assets/urdf/project_mobile_robot/project_mobile_robot.urdf.xacro (robot description, xacro)
@@ -57,11 +57,11 @@
     </joint>
   </xacro:macro>
-  <xacro:wheel_link name="left" linkrpy="0 0 0" axisxyz="1 0 0" originxyz="0.15 0 -0.075"/>
-  <xacro:wheel_link name="right" linkrpy="0 0 0" axisxyz="1 0 0" originxyz="-0.15 0 -0.075"/>
-  <xacro:wheel_link name="front" linkrpy="0 0 0" axisxyz="0 1 0" originxyz="0 0.15 -0.075"/>
-  <xacro:wheel_link name="back" linkrpy="0 0 0" axisxyz="0 1 0" originxyz="0 -0.15 -0.075"/>
+  <xacro:wheel_link name="front_right" linkrpy="0 0 0" axisxyz="1 0 0" originxyz="0.15 0 -0.075"/>
+  <xacro:wheel_link name="back_left" linkrpy="0 0 0" axisxyz="1 0 0" originxyz="-0.15 0 -0.075"/>
+  <xacro:wheel_link name="front_left" linkrpy="0 0 0" axisxyz="0 1 0" originxyz="0 0.15 -0.075"/>
+  <xacro:wheel_link name="back_right" linkrpy="0 0 0" axisxyz="0 1 0" originxyz="0 -0.15 -0.075"/>
   <!-- Lidar sensor -->
   <xacro:include filename="lidar_sensor.urdf.xacro"/>
-  <!--Q:ray_count_horizontal=10, DQN:ray_count_horizontal=216 -->
+  <!--Q:ray_count_horizontal=60, DQN:ray_count_horizontal=216 -->
   <xacro:lidar_sensor
     name="sonar"
@@ -73,7 +73,7 @@
     field_of_view_horizontal="${270*M_PI/180}"
     field_of_view_vertical="${1*M_PI/180}"
-    ray_count_horizontal="2162"
+    ray_count_horizontal="62"
     ray_count_vertical="1">
-    <origin xyz="0 0.0 0.1" rpy="0 0 0"/>
+    <origin xyz="0 0.0 0.1" rpy="0 0 ${M_PI/4}"/>
   </xacro:lidar_sensor>
   <gazebo>
